File: pcbs/keyboard/src/Keyboard _Board.brd (EAGLE design)
At the start: 320 x 136 mm, 292 parts, among them J1 M55-6001242R, J2 M55-6001242R, J3 1-1775333-6CONN16_1-1775333-6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, J4 F31L-1A7H1-11012, U1 SC0914(13), U2 AP2112K-3.3TRG1SOT_RG1_DIO, U3 W25Q128JVSIM_TR, U4 SN74AHCT1G125DBVR, U5 SN74AHCT1G125DBVR, Y1 ABM8-272-T3

Commit message: fix: repair CMDeck Rev A PCB defects
Connections:
- removed net N$12: R4.1, R6.2, U3.1
- new net QSPI_SS_N: R4.1, R6.2, U1.56, U3.1
Routing:
- net QSPI_SS_N: track 0.00 -> 36.7 mm
- net N$12: track 4.54 -> 0.00 mm
Changed lines of the file:
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@@
 <wire x1="164.368725" y1="121.32" x2="163.455" y2="121.32" width="0.2032" layer="16"/>
 </signal>
-<signal name="N$12">
+<signal name="QSPI_SS_N">
+<contactref element="U1" pad="56"/>
 <contactref element="U3" pad="1"/>
 <contactref element="R4" pad="1"/>
@@
 <wire x1="180.0555" y1="119.38" x2="180.135" y2="119.3005" width="0.2032" layer="16"/>
 <wire x1="180.135" y1="119.3005" x2="180.135" y2="116.84" width="0.2032" layer="16"/>
+<wire x1="163.455" y1="119.32" x2="163.8106" y2="119.32" width="0.2032" layer="16"/>
+<wire x1="163.8106" y1="119.32" x2="166.1616" y2="116.969" width="0.2032" layer="16"/>
+<wire x1="166.1616" y1="116.969" x2="168.10935" y2="116.969" width="0.2032" layer="16"/>
+<wire x1="168.10935" y1="116.969" x2="168.9354" y2="116.14295" width="0.2032" layer="16"/>
+<wire x1="168.9354" y1="116.14295" x2="168.9354" y2="113.1367" width="0.2032" layer="16"/>
+<wire x1="168.9354" y1="113.1367" x2="171.0233" y2="111.0488" width="0.2032" layer="16"/>
+<wire x1="171.0233" y1="111.0488" x2="181.96425" y2="111.0488" width="0.2032" layer="16"/>
+<wire x1="181.96425" y1="111.0488" x2="183.0832" y2="112.16775" width="0.2032" layer="16"/>
+<wire x1="183.0832" y1="112.16775" x2="183.0832" y2="115.57" width="0.2032" layer="16"/>
+<wire x1="183.0832" y1="115.57" x2="181.8132" y2="116.84" width="0.2032" layer="16"/>
+<wire x1="181.8132" y1="116.84" x2="180.135" y2="116.84" width="0.2032" layer="16"/>
 </signal>
 <signal name="!RESET">
