File: pcbs/keyboard/src/Keyboard _Schematic.sch (EAGLE design)
At the start: 292 parts, among them J1 M55-6001242R, J2 M55-6001242R, J3 1-1775333-6CONN16_1-1775333-6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, J4 F31L-1A7H1-11012, U1 SC0914(13), U2 AP2112K-3.3TRG1SOT_RG1_DIO, U3 W25Q128JVSIM_TR, U4 SN74AHCT1G125DBVR, U5 SN74AHCT1G125DBVR, Y1 ABM8-272-T3

Commit message: fix: repair CMDeck Rev A PCB defects
Connections:
- removed net N$12: R4.1, R6.2, U3.!CS
- new net QSPI_SS_N: R4.1, R6.2, U1.QSPI_SS_N, U3.!CS
Changed lines of the file:
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@@
 </segment>
 </net>
-<net name="N$12" class="0">
+<net name="QSPI_SS_N" class="0">
+<segment>
+<pinref part="U1" gate="G$1" pin="QSPI_SS_N"/>
+<wire x1="106.68" y1="101.6" x2="109.22" y2="101.6" width="0.1524" layer="91"/>
+<label x="109.22" y="101.6" size="1.27" layer="95" xref="yes"/>
+</segment>
 <segment>
 <pinref part="U3" gate="G$1" pin="!CS"/>
