File: pcbs/main board/src/Main Board _Board.brd (EAGLE design)
At the start: 320 x 56 mm, 149 parts, among them IC1 TPA6132A2, J1 FH12-22S-0.5SH(55)CONN_FH12-2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, J10 L8BE-1G1T-BFH, J11 UJ20-C-R-G-TH-2-P14-TR, J12 S2B-XH-A, J13 S2B-XH-A, J14 2328702-8, J16 M55-7011242R, J17 SJ-3579AN, J18 61201621721, J19 61201621721, J2 HD05-19-TH-TR, J21 M55-7011242R, J3 HD05-19-TH-TR, J4 614104190121, J5 UJ20-C-R-G-TH-2-P14-TR, J6 UJ20-C-R-G-TH-2-P14-TR, J7 1-2199119-5, J8 SM04B-SRSS-TBCONN_SM04B-SRSS-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, J9 UJ20-C-R-G-TH-2-P14-TR, U1 CM5108064B, U10 TPD4EUSB30DQAR, U11 TPD4EUSB30DQAR, U12 AP3441SHE-7BIC8_AP3441SHE-7B_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, U13 PCM5100APWRPW0020A, U14 MAX98306ETD+T, U2 RT9742SNGVSOT_42SNGV_RIT, U3 AP22653W6-7, U4 USB2514B/M2SQFN36_6X6_MCH, U5 FSUSB42MUX, U6 TPD4EUSB30DQAR, U7 TPD4EUSB30DQAR, U8 TPD4EUSB30DQAR, U9 TPD4EUSB30DQAR, Y1 24 MHz, Y2 ASEK-32.768KHZ-L-R-T

Commit message: fix: repair CMDeck Rev A PCB defects
Parts:
- added JP5: DSI 3V3 OPEN, CMDeck-Jumpers:SJ_2_NO
- added TP15, TP16: TPPAD1-13, testpad:P1-13
Connections:
- new net DSI_3V3: J1.22, JP5.2
- net CM5_3.3V: now also JP5.1; no longer J1.22
- net GND: now also TP16.TP
- net PWR_BUTTON: now also TP15.TP
Routing:
- net CM5_3.3V: track 602.9 -> 599.5 mm
- net DSI_3V3: track 0.00 -> 1.92 mm
- net PWR_BUTTON: vias 5 -> 4
Other:
- board text added: "PWR"
- board text added: "X1203 BTN"
Changed lines of the file:
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@@
 <vertex x="315.39256875" y="27.8030875"/>
 </polygon>
+<text x="63.5" y="36.3" size="0.8128" layer="21" ratio="12">X1203 BTN</text>
+<text x="64.65" y="31.3" size="0.6096" layer="21" ratio="12">PWR</text>
+<text x="68.05" y="31.3" size="0.6096" layer="21" ratio="12">GND</text>
 </plain>
 <attributes>
@@
 <attribute name="VALUE" x="19.05" y="50.673" size="0.0254" layer="27"/>
 </element>
+<element name="TP15" library="testpad" library_urn="urn:adsk.eagle:library:385" package="P1-13" value="TPPAD1-13" x="66.04" y="33.655" smashed="yes">
+<attribute name="NAME" x="65.024" y="34.925" size="0.8128" layer="25" ratio="12"/>
+<attribute name="TP_SIGNAL_NAME" value="PWR_BUTTON" x="64.77" y="31.115" size="1" layer="37"/>
+<attribute name="VALUE" x="66.04" y="33.655" size="0.0254" layer="27"/>
+</element>
+<element name="TP16" library="testpad" library_urn="urn:adsk.eagle:library:385" package="P1-13" value="TPPAD1-13" x="68.84" y="33.655" smashed="yes">
+<attribute name="NAME" x="67.824" y="34.925" size="0.8128" layer="25" ratio="12"/>
+<attribute name="TP_SIGNAL_NAME" value="GND" x="67.57" y="31.115" size="1" layer="37"/>
+<attribute name="VALUE" x="68.84" y="33.655" size="0.0254" layer="27"/>
+</element>
+<element name="JP5" library="CMDeck-Jumpers" package="SJ_2_NO" value="DSI 3V3 OPEN" x="181.94" y="46.4796" smashed="yes">
+<attribute name="NAME" x="180.49" y="47.5296" size="0.8128" layer="25" ratio="12"/>
+<attribute name="VALUE" x="180.49" y="44.6296" size="0.8128" layer="27" display="off"/>
+</element>
 </elements>
 <signals>
 <signal name="GND">
+<contactref element="TP16" pad="TP"/>
 <contactref element="U1" pad="1"/>
 <contactref element="U1" pad="2"/>
@@
 <contactref element="U1" pad="84"/>
 <contactref element="U1" pad="86"/>
-<contactref element="J1" pad="22"/>
+<contactref element="JP5" pad="1"/>
 <contactref element="U5" pad="1"/>
 <contactref element="C3" pad="1"/>
@@
 <via x="159.6898" y="18.7452" extent="1-16" drill="0.3">
 </via>
-<wire x1="184.6128" y1="46.4796" x2="164.5896" y2="46.4796" width="0.1524" layer="1"/>
+<wire x1="181.19" y1="46.4796" x2="164.5896" y2="46.4796" width="0.1524" layer="1"/>
 <wire x1="164.5896" y1="46.4796" x2="164.465" y2="46.355" width="0.1524" layer="1"/>
 <via x="164.465" y="46.355" extent="1-16" drill="0.3">
@@
 <wire x1="281.94" y1="47.6686" x2="282.575" y2="47.6686" width="0.1524" layer="16"/>
 </signal>
+<signal name="DSI_3V3">
+<contactref element="JP5" pad="2"/>
+<contactref element="J1" pad="22"/>
+<wire x1="182.69" y1="46.4796" x2="184.6128" y2="46.4796" width="0.1524" layer="1"/>
+</signal>
 <signal name="PWR_BUTTON">
+<contactref element="TP15" pad="TP"/>
 <contactref element="U1" pad="92"/>
 <contactref element="U$1" pad="PWR_SW"/>
@@
 <wire x1="68.4022" y1="37.4142" x2="66.04" y2="35.052" width="0.2032" layer="1"/>
 <wire x1="66.04" y1="35.052" x2="66.04" y2="33.655" width="0.2032" layer="1"/>
-<via x="66.04" y="33.655" extent="1-16" drill="0.35">
-</via>
 <wire x1="65.6516" y1="33.2666" x2="66.04" y2="33.655" width="0.2032" layer="16"/>
 <wire x1="65.6516" y1="30.62791875" x2="65.6516" y2="33.2666" width="0.2032" layer="16"/>
