File: pcbs/main board/src/Main_Board_Schematic.sch (EAGLE design)
At the start: 149 parts, among them IC1 TPA6132A2, J1 FH12-22S-0.5SH(55)CONN_FH12-2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, J10 L8BE-1G1T-BFH, J11 UJ20-C-R-G-TH-2-P14-TR, J12 S2B-XH-A, J13 S2B-XH-A, J14 2328702-8, J16 M55-7011242R, J17 SJ-3579AN, J18 61201621721, J19 61201621721, J2 HD05-19-TH-TR, J21 M55-7011242R, J3 HD05-19-TH-TR, J4 614104190121, J5 UJ20-C-R-G-TH-2-P14-TR, J6 UJ20-C-R-G-TH-2-P14-TR, J7 1-2199119-5, J8 SM04B-SRSS-TBCONN_SM04B-SRSS-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, J9 UJ20-C-R-G-TH-2-P14-TR, U1 CM5108064B, U10 TPD4EUSB30DQAR, U11 TPD4EUSB30DQAR, U12 AP3441SHE-7BIC8_AP3441SHE-7B_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, U13 PCM5100APWRPW0020A, U14 MAX98306ETD+T, U2 RT9742SNGVSOT_42SNGV_RIT, U3 AP22653W6-7, U4 USB2514B/M2SQFN36_6X6_MCH, U5 FSUSB42MUX, U6 TPD4EUSB30DQAR, U7 TPD4EUSB30DQAR, U8 TPD4EUSB30DQAR, U9 TPD4EUSB30DQAR, Y1 24 MHz, Y2 ASEK-32.768KHZ-L-R-T

Commit message: fix: repair CMDeck Rev A PCB defects
Parts:
- added JP5: DSI 3V3 OPEN, CMDeck-Jumpers:SJ_2_NO
- added TP15, TP16: TPPAD1-13, testpad:TPPAD1-13
Connections:
- new net DSI_3V3: J1.22, JP5.2
- net CM5_3.3V: now also JP5.1; no longer J1.22
- net GND: now also TP16.TP
- net PWR_BUTTON: now also TP15.TP
Changed lines of the file:
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@@
 <part name="TP13" library="testpad" library_urn="urn:adsk.eagle:library:385" deviceset="TP" device="B1,27" package3d_urn="urn:adsk.eagle:package:27944/2" value="TPB1,27"/>
 <part name="TP14" library="testpad" library_urn="urn:adsk.eagle:library:385" deviceset="TP" device="B1,27" package3d_urn="urn:adsk.eagle:package:27944/2" value="TPB1,27"/>
+<part name="TP15" library="testpad" library_urn="urn:adsk.eagle:library:385" deviceset="TP" device="PAD1-13" value="TPPAD1-13"/>
+<part name="TP16" library="testpad" library_urn="urn:adsk.eagle:library:385" deviceset="TP" device="PAD1-13" value="TPPAD1-13"/>
+<part name="JP5" library="CMDeck-Jumpers" deviceset="SJ_2_NO" device="" value="DSI 3V3 OPEN"/>
 </parts>
 <sheets>
@@
 <attribute name="NAME" x="235.3046" y="175.4886" size="2.083" layer="95" ratio="6"/>
 </instance>
+<instance part="JP5" gate="G$1" x="220.98" y="116.84" smashed="yes" grouprefs="DSI_CSI_CONNECTOR">
+<attribute name="NAME" x="218.44" y="118.11" size="1.27" layer="95"/>
+<attribute name="VALUE" x="218.44" y="114.3" size="1.27" layer="96"/>
+</instance>
 <instance part="J2" gate="G$1" x="53.34" y="127" smashed="yes" grouprefs="HDMI_0">
 <attribute name="NAME" x="38.1" y="165.862" size="1.778" layer="95"/>
@@
 <net name="CM5_3.3V" class="0">
 <segment>
-<wire x1="231.14" y1="116.84" x2="187.96" y2="116.84" width="0.1524" layer="91" grouprefs="DSI_CSI_CONNECTOR"/>
+<wire x1="215.9" y1="116.84" x2="187.96" y2="116.84" width="0.1524" layer="91" grouprefs="DSI_CSI_CONNECTOR"/>
 <label x="187.96" y="116.84" size="1.27" layer="95" rot="R180" xref="yes" grouprefs="DSI_CSI_CONNECTOR"/>
+<pinref part="JP5" gate="G$1" pin="1"/>
+</segment>
+</net>
+<net name="DSI_3V3" class="0">
+<segment>
+<pinref part="JP5" gate="G$1" pin="2"/>
+<wire x1="226.06" y1="116.84" x2="231.14" y2="116.84" width="0.1524" layer="91" grouprefs="DSI_CSI_CONNECTOR"/>
 <pinref part="J1" gate="A" pin="22"/>
 </segment>
@@
 <attribute name="TP_SIGNAL_NAME" x="52.07" y="140.97" size="1.778" layer="97" rot="R90"/>
 </instance>
+<instance part="TP15" gate="G$1" x="124.46" y="144.78" smashed="yes">
+<attribute name="NAME" x="121.92" y="146.05" size="1.27" layer="95"/>
+<attribute name="TP_SIGNAL_NAME" value="PWR_BUTTON" x="125.73" y="143.51" size="1.27" layer="97"/>
+</instance>
+<instance part="TP16" gate="G$1" x="137.16" y="144.78" smashed="yes">
+<attribute name="NAME" x="134.62" y="146.05" size="1.27" layer="95"/>
+<attribute name="TP_SIGNAL_NAME" value="GND" x="138.43" y="143.51" size="1.27" layer="97"/>
+</instance>
 </instances>
 <busses>
@@
 </segment>
 <segment>
+<pinref part="TP16" gate="G$1" pin="TP"/>
+<wire x1="137.16" y1="142.24" x2="142.24" y2="142.24" width="0.1524" layer="91"/>
+<label x="142.24" y="142.24" size="1.27" layer="95" xref="yes"/>
+</segment>
+<segment>
 <pinref part="SUPPLY60" gate="G$1" pin="GND"/>
 <wire x1="162.56" y1="142.24" x2="162.56" y2="147.32" width="0.1524" layer="91" grouprefs="5V_IN"/>
@@
 <pinref part="J16" gate="G$1" pin="B3"/>
 </segment>
+<segment>
+<pinref part="TP15" gate="G$1" pin="TP"/>
+<wire x1="124.46" y1="142.24" x2="129.54" y2="142.24" width="0.1524" layer="91"/>
+<label x="129.54" y="142.24" size="1.27" layer="95" xref="yes"/>
+</segment>
 </net>
